File: kicad/adapter-u6w5.sch (KiCad schematic (older format))
At the start: 4 parts, among them J1 THUMB_RIGHT_SPC_KB600, J5 THUMB_LEFT_BAK, J6 THUMB_RIGHT_SPC, J8 THUMB_LEFT_BAK_KB600

Commit message: route
Connections:
- net COL_5 renamed COL_5_L
- net COL_5_L: no longer J1.8 (Pin_8), J6.8 (Pin_8)
- net COL_6 renamed COL_6_L
- net COL_6_L: no longer J1.7 (Pin_7), J6.7 (Pin_7)
- net ROW_2 renamed ROW_2_L
- net ROW_3 renamed ROW_3_L
- net ROW_4 renamed ROW_4_L
- net ROW_5 renamed ROW_5_L
- net ROW_6 renamed ROW_6_R
- net ROW_7 renamed ROW_7_R
- net ROW_8 renamed ROW_8_R
- net ROW_9 renamed ROW_9_R
- new net COL_5_R: J1.8 (Pin_8), J6.8 (Pin_8)
- new net COL_6_R: J1.7 (Pin_7), J6.7 (Pin_7)
Changed lines of the file:
@@
 NoConn ~ 10100 5650
 Text Label 9750 4750 0    50   ~ 10
-ROW_4
+ROW_4_L
 Text Label 9750 4950 0    50   ~ 10
-ROW_5
+ROW_5_L
 $Comp
 L Connector_Generic:Conn_01x10 J5
@@
 $EndComp
 Text Label 9750 5450 0    50   ~ 10
-ROW_3
+ROW_3_L
 Text Label 9750 5150 0    50   ~ 0
-COL_5
+COL_5_L
 Text Label 9750 5050 0    50   ~ 0
-COL_6
+COL_6_L
 Text Label 1900 5250 2    50   ~ 10
-ROW_9
+ROW_9_R
 Wire Wire Line
 	1900 5250 1600 5250
 Text Label 1900 5350 2    50   ~ 0
-COL_6
+COL_6_R
 Wire Wire Line
 	1600 5350 1900 5350
 Text Label 1900 5450 2    50   ~ 0
-COL_5
+COL_5_R
 Wire Wire Line
 	1900 5450 1600 5450
 Text Label 1900 5150 2    50   ~ 0
-ROW_8
+ROW_8_R
 Wire Wire Line
 	1900 5150 1600 5150
 Text Label 1900 5050 2    50   ~ 0
-ROW_7
+ROW_7_R
 Wire Wire Line
 	1900 5050 1600 5050
 Text Label 1900 4950 2    50   ~ 10
-ROW_6
+ROW_6_R
 Wire Wire Line
 	1900 4950 1600 4950
 Text Label 9750 4850 0    50   ~ 10
-ROW_2
+ROW_2_L
 Wire Wire Line
 	9750 4750 10100 4750
@@
 NoConn ~ 3350 5750
 Text Label 3650 5250 2    50   ~ 10
-ROW_9
+ROW_9_R
 Wire Wire Line
 	3650 5450 3350 5450
 Text Label 3650 5350 2    50   ~ 0
-COL_6
+COL_6_R
 Text Label 3650 5450 2    50   ~ 0
-COL_5
+COL_5_R
 Text Label 3650 5150 2    50   ~ 0
-ROW_8
+ROW_8_R
 Wire Wire Line
 	3650 5350 3350 5350
 Text Label 3650 5050 2    50   ~ 0
-ROW_7
+ROW_7_R
 Wire Wire Line
 	3650 5250 3350 5250
 Text Label 3650 4950 2    50   ~ 10
-ROW_6
+ROW_6_R
 Wire Wire Line
 	3650 5150 3350 5150
@@
 NoConn ~ 8350 5850
 Text Label 8000 4750 0    50   ~ 10
-ROW_4
+ROW_4_L
 Text Label 8000 4950 0    50   ~ 10
-ROW_5
+ROW_5_L
 $Comp
 L Connector_Generic:Conn_01x13 J8
@@
 $EndComp
 Text Label 8000 5450 0    50   ~ 10
-ROW_3
+ROW_3_L
 Text Label 8000 5150 0    50   ~ 0
-COL_5
+COL_5_L
 Text Label 8000 5050 0    50   ~ 0
-COL_6
+COL_6_L
 Text Label 8000 4850 0    50   ~ 10
-ROW_2
+ROW_2_L
 Wire Wire Line
 	8000 4750 8350 4750
